Commit message: M1-M7 模块开发：仿真环境、导航集成、巡逻序列、电池回充、视觉对接、轮次调度、异常处理
M1: 仿真环境与基础移动（模型/世界/键盘遥控/里程计TF/RViz2）
M2: Nav2 导航集成（静态地图/参数配置/动作客户端/动态避障）
M3: 巡逻序列实现（行为树节点/waypoints/堵赛放弃/断点续巡）
M4: 电池模拟与低电回充（充放电模拟/低电中断/充电恢复）
M5: 视觉分段对接（视觉伺服P控制器/重试机制/对接充电）
M6: 轮次调度与完整任务编排（轮次循环/待命点/断点恢复/索引重置）
M7: 异常处理与日志（报警节点/堵赛/对接失败/电池超时/定位丢失检测）

File: patrol_robot_ws/src/nav2_demo/models/patrol_bot/model.urdf (robot description, URDF)
Before this commit: robot patrol_bot, 4 links, 3 joints
Links:
- added link camera_link
Joints:
- added joint camera_joint: type fixed, parent base_link, child camera_link, origin xyz=0.18 0 0.12 rpy=0 0 0
