Commit message: 修复 Gazebo/ROS2 坐标不一致及仿真架构重构
- 移除 patrol_simulation.launch.py 中与 AMCL 冲突的静态 map→odom TF
- AMCL 加入 lifecycle_manager 自动激活列表
- 新增 odom_bridge.py 替代 odom_republisher，可配置帧名桥接
- SDF: 移除 base_footprint 回归原物理根 link 结构，修复 caster 碰撞体高度
- SDF: 翻转驱动轮关节轴 0→-1 修复物理运动方向与里程计符号不一致
- URDF: 清理 Gazebo 插件，SDF 独立管理仿真物理
- pointcloud_to_scan: 输入 topic 可配置参数

Co-Authored-By: Claude Opus 4.7 <noreply@anthropic.com>

File: patrol_robot_ws/src/patrol_bot/models/patrol_bot/model.urdf (robot description, URDF)
Before this commit: robot patrol_bot, 5 links, 4 joints
Links:
- removed link chassis
- added link caster; visual sphere radius=0.03
- added link left_wheel; visual cylinder length=0.02 radius=0.05
- added link right_wheel; visual cylinder length=0.02 radius=0.05
- link base_link: geometry visual box size=0.4 0.3 0.15
- link camera_link: geometry visual box size=0.03 0.03 0.02
- link lidar_link: geometry visual cylinder length=0.04 radius=0.04
Joints:
- removed joint chassis_joint
- added joint caster_joint: type fixed, parent base_link, child caster, origin xyz=-0.15 0 -0.14 rpy=0 0 0
- added joint left_wheel_joint: type continuous, parent base_link, child left_wheel, origin xyz=0.12 0.18 -0.12 rpy=0 0 0, axis 0 1 0
- added joint right_wheel_joint: type continuous, parent base_link, child right_wheel, origin xyz=0.12 -0.18 -0.12 rpy=0 0 0, axis 0 1 0
